File: DMH_CV_Mixer_PANEL/DMH_CV_Mixer_PANEL.kicad_sch (KiCad schematic)
At the start: 25 parts, among them J0 Panel_GND_Solder_Wire_Pad

Commit message: Panel design done
Parts:
- H10: value CV C Amt -> In C2
- H12: value Offset B -> In B1; footprint SynthStuff:Pot_Cutout_Tiny -> SynthStuff:Pot_Cutout_Tiny_attv_P110KH1
- H13: value CV B Amt -> In B2
- H14: value In C -> In C1
- H15: value In B -> In B1
- H17: value CV B -> In B2
- H18: value CV C -> In C2
- H19: value Offset D -> In D1; footprint SynthStuff:Pot_Cutout_Tiny -> SynthStuff:Pot_Cutout_Tiny_attv_P110KH1
- H20: value CV D Amt -> In D2
- H21: value In D -> In D1
- H22: value CV D -> In D2
- H5: value Offset A -> In A1; footprint SynthStuff:Pot_Cutout_Tiny -> SynthStuff:Pot_Cutout_Tiny_attv_P110KH1
- H6: value CV A Amt -> In A2
- H7: value Offset C -> In C1; footprint SynthStuff:Pot_Cutout_Tiny -> SynthStuff:Pot_Cutout_Tiny_attv_P110KH1
- H8: value In A -> In A1
- H9: value CV A -> In A2
Changed lines of the file:
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@@
 			)
 		)
-		(property "Value" "Offset C"
+		(property "Value" "In C1"
 			(at 104.14 88.8999 0)
 			(effects
@@
 			)
 		)
-		(property "Footprint" "SynthStuff:Pot_Cutout_Tiny"
+		(property "Footprint" "SynthStuff:Pot_Cutout_Tiny_attv_P110KH1"
 			(at 101.6 90.17 0)
 			(effects
@@
 			)
 		)
-		(property "Value" "CV B"
+		(property "Value" "In B2"
 			(at 40.64 215.8999 0)
 			(effects
@@
 			)
 		)
-		(property "Value" "CV C"
+		(property "Value" "In C2"
 			(at 104.14 139.6999 0)
 			(effects
@@
 			)
 		)
-		(property "Value" "Offset A"
+		(property "Value" "In A1"
 			(at 40.64 88.8999 0)
 			(effects
@@
 			)
 		)
-		(property "Footprint" "SynthStuff:Pot_Cutout_Tiny"
+		(property "Footprint" "SynthStuff:Pot_Cutout_Tiny_attv_P110KH1"
 			(at 38.1 90.17 0)
 			(effects
@@
 			)
 		)
-		(property "Value" "In A"
+		(property "Value" "In A1"
 			(at 40.64 126.9999 0)
 			(effects
@@
 			)
 		)
-		(property "Value" "CV D Amt"
+		(property "Value" "In D2"
 			(at 104.14 177.7999 0)
 			(effects
@@
 			)
 		)
-		(property "Value" "CV A"
+		(property "Value" "In A2"
 			(at 40.64 139.6999 0)
 			(effects
@@
 			)
 		)
-		(property "Value" "Offset D"
+		(property "Value" "In D1"
 			(at 104.14 165.0999 0)
 			(effects
@@
 			)
 		)
-		(property "Footprint" "SynthStuff:Pot_Cutout_Tiny"
+		(property "Footprint" "SynthStuff:Pot_Cutout_Tiny_attv_P110KH1"
 			(at 101.6 166.37 0)
 			(effects
@@
 			)
 		)
-		(property "Value" "In C"
+		(property "Value" "In C1"
 			(at 104.14 126.9999 0)
 			(effects
@@
 			)
 		)
-		(property "Value" "CV C Amt"
+		(property "Value" "In C2"
 			(at 104.14 101.5999 0)
 			(effects
@@
 			)
 		)
-		(property "Value" "In B"
+		(property "Value" "In B1"
 			(at 40.64 203.1999 0)
 			(effects
@@
 			)
 		)
-		(property "Value" "CV D"
+		(property "Value" "In D2"
 			(at 104.14 215.8999 0)
 			(effects
@@
 			)
 		)
-		(property "Value" "In D"
+		(property "Value" "In D1"
 			(at 104.14 203.1999 0)
 			(effects
@@
 			)
 		)
-		(property "Value" "CV A Amt"
+		(property "Value" "In A2"
 			(at 40.64 101.5999 0)
 			(effects
@@
 			)
 		)
-		(property "Value" "CV B Amt"
+		(property "Value" "In B2"
 			(at 40.64 177.7999 0)
 			(effects
@@
 			)
 		)
-		(property "Value" "Offset B"
+		(property "Value" "In B1"
 			(at 40.64 165.0999 0)
 			(effects
@@
 			)
 		)
-		(property "Footprint" "SynthStuff:Pot_Cutout_Tiny"
+		(property "Footprint" "SynthStuff:Pot_Cutout_Tiny_attv_P110KH1"
 			(at 38.1 166.37 0)
 			(effects
