File: DMH_CV_Mixer_PCB_1/Core_Circuit.kicad_sch (KiCad schematic)
At the start: 0 parts

Commit message: Finished IO page
Parts:
- added R1: 33k, Resistor_THT:R_Axial_DIN0207_L6.3mm_D2.5mm_P7.62mm_Horizontal, symbol Device:R_US
- added RV1: 50k, Potentiometer_THT:Potentiometer_Bourns_3296X_Horizontal, symbol Device:R_Potentiometer_Trim_US
- added RV2: 100k, SynthStuff:Potentiometer_TT_P110KH1, symbol Device:R_Potentiometer_US
- added U1: TL074, Package_DIP:DIP-14_W7.62mm_Socket, symbol Amplifier_Operational:TL074
Connections:
- new net: RV1.2, RV1.3, U1.1
- new net: R1.2, RV1.1, U1.2 (-)
- new net: RV2.2, U1.3 (+)
- new net: R1.1, RV2.3
- new net GND: RV2.1
