File: DMH_CV_Mixer_PCB_1/Core_Circuit.kicad_sch (KiCad schematic)
At the start: 4 parts, among them U1 TL074

Commit message: Schematic in progress
Parts:
- added R10, R11, R12, R13, R14, R15, R16, R17, R18, R19, R20, R21, R22, R23, R24, R25, R26, R27, R28, R29, R30, R31, R9: 100k, Resistor_THT:R_Axial_DIN0207_L6.3mm_D2.5mm_P7.62mm_Horizontal, symbol Device:R_US
- added R2, R3, R4, R5, R6, R7, R8: 33k, Resistor_THT:R_Axial_DIN0207_L6.3mm_D2.5mm_P7.62mm_Horizontal, symbol Device:R_US
- added RV10, RV12, RV14, RV16, RV4, RV6, RV8: 100k, SynthStuff:Potentiometer_TT_P110KH1, symbol Device:R_Potentiometer_US
- added RV11, RV13, RV15, RV3, RV5, RV7, RV9: 50k, Potentiometer_THT:Potentiometer_Bourns_3296X_Horizontal, symbol Device:R_Potentiometer_Trim_US
- added U10, U11, U12, U13, U14, U15, U16, U9: TL074, symbol Amplifier_Operational:TL074
- added U2, U3, U4, U5, U6, U7, U8: TL074, Package_DIP:DIP-14_W7.62mm_Socket, symbol Amplifier_Operational:TL074
- RV1: Function CV A1 Zero -> A1 Zero
- RV2: Function CV A1 Amt -> A1 Amt
Connections:
- net GND: now also RV10.1, RV12.1, RV14.1, RV16.1, RV4.1, RV6.1, RV8.1, U10.3 (+), U11.3 (+), U12.3 (+), U13.3 (+), U14.3 (+), U15.3 (+), U16.3 (+), U9.3 (+)
- net at RV1.2, RV1.3, U1.1: now also R9.1
- net A In 1: now reaches R1.1, RV2.3
- new net: R24.2, R27.1, U15.1
- new net: R25.1, R27.2, U16.2 (-)
- new net: R11.2, R12.1, U9.1
- new net: R10.2, R11.1, R9.2, U9.2 (-)
- new net: R16.1, RV3.2, RV3.3, U2.1
- new net: R2.2, RV3.1, U2.2 (-)
- new net: RV4.2, U2.3 (+)
- new net: R19.2, R22.1, U13.1
- new net: R19.1, R21.2, R23.2, R30.2, U13.2 (-)
- new net: R21.1, RV5.2, RV5.3, U3.1
- new net: R3.2, RV5.1, U3.2 (-)
- new net: RV6.2, U3.3 (+)
- new net: R8.2, RV15.1, U8.2 (-)
- new net: R28.1, RV15.2, RV15.3, U8.1
- new net: R12.2, R13.1, U10.2 (-)
- new net: R5.2, RV9.1, U5.2 (-)
- new net: R10.1, RV9.2, RV9.3, U5.1
- new net: RV10.2, U5.3 (+)
- new net: R24.1, R26.2, R28.2, R31.2, U15.2 (-)
- new net: R20.1, R22.2, U14.2 (-)
- new net: R14.1, R16.2, R18.2, R29.2, U11.2 (-)
- new net: R6.2, RV11.1, U6.2 (-)
- new net: R18.1, RV11.2, RV11.3, U6.1
- new net: RV12.2, U6.3 (+)
- new net: R4.2, RV7.1, U4.2 (-)
- new net: R26.1, RV7.2, RV7.3, U4.1
- new net: R14.2, R17.1, U11.1
- new net: R15.1, R17.2, U12.2 (-)
- new net: RV16.2, U8.3 (+)
- new net: RV8.2, U4.3 (+)
- new net: R23.1, RV13.2, RV13.3, U7.1
- new net: R7.2, RV13.1, U7.2 (-)
- new net: RV14.2, U7.3 (+)
- new net A In 2: R5.1, RV10.3
- new net B In 1: R2.1, RV4.3
- new net B In 2: R6.1, RV12.3
- new net C In 1: R3.1, RV6.3
- new net C In 2: R7.1, RV14.3
- new net D In 1: R4.1, RV8.3
- new net D In 2: R8.1, RV16.3
- new net In AB: R29.1
- new net In BC: R30.1
- new net In CD: R31.1
- new net Out A: R13.2, U10.1
- new net Out B: R15.2, U12.1
- new net Out C: R20.2, U14.1
- new net Out D: R25.2, U16.1
Other:
- moved on the sheet: R1, RV1, RV2, U1A
