File: DMH_CV_Mixer_PCB_1/DMH_CV_Mixer_PCB_1.kicad_sch (KiCad schematic)
At the start: 0 parts

Commit message: Schematic in progress
Other:
- sheet Core Circuit ports: added A In 1, A In 2, B In 1, B In 2, C In 1, C In 2, D In 1, D In 2, In AB, In BC, In CD, Out A, Out B, Out C, Out D; removed none
- sheet Inputs and Outputs ports: added In A1 Jack, In A2 Jack, In B1 Jack, In B2 Jack, In C1 Jack, In C2 Jack, In D1 Jack, In D2 Jack, Out A Jack, Out A Jack TN, Out B Jack, Out B Jack TN, Out C Jack, Out C Jack TN, Out D Jack, Out D Jack TN; removed none
